File: hardware/Shunt_Buddy.kicad_pcb (KiCad board)
At the start: 2 copper layers, 50 x 50 mm, 38 parts, among them J1 USB_C_Receptacle_USB2.0_16P, J2 Conn_Coaxial, J3 Screw_Terminal_01x03, J4 Conn_01x03, J5 Conn_01x03, SW1 SW_DIP_x05, U1 INA225, U2 MIC5205-4.0YM5, U3 MCP6L01x-xOT

Commit message: Cleanups
Routing:
- net /IN+: track 23.0 -> 2.42 mm
- net /IN-: track 21.2 -> 2.42 mm
- net GND: track 22.7 -> 27.1 mm, vias 72 -> 81
- added copper zone on F.Cu, net /IN+
- added copper zone on F.Cu, net /IN-
